File: CARDIO-TUNE/HARDWARE/CARDIO_TUNE/CARDIO_TUNE.kicad_pcb (KiCad board)
At the start: 2 copper layers, 13 parts, among them J1 TPA, J2 MAX30102, J3 Screw_Terminal_01x02, SW1 SW_Nidec_CAS-120A1, SW2 SW_Push, U1 ESP32-DEVKITC

Commit message: Add files via upload
Parts:
- added G***: LOGO, HUELLAS:cardiotune, F.Cu at (47.0, 64.5)
- added G***: LOGO, HUELLAS:mollourtadopaty, F.Cu at (44.6, 66.1)
- added R5: 220, Resistor_THT:R_Axial_DIN0207_L6.3mm_D2.5mm_P7.62mm_Horizontal, F.Cu at (85.5, 70.3)
- J1: value TPA -> TRRS
- SW1: footprint Button_Switch_SMD:Nidec_Copal_CAS-120A -> Connector_PinHeader_2.54mm:PinHeader_2x01_P2.54mm_Vertical
- moved D1 57.2 mm to (29.5, 62.3), turned to 0 degrees
- moved R3 46.6 mm to (32.0, 66.8), turned to 180 degrees
- moved SW1 41.9 mm to (30.2, 71.1), turned to 0 degrees
- moved U3 35.4 mm to (41.5, 44.3)
- moved J1 33.9 mm to (28.0, 38.0), turned to 0 degrees
- moved U1 30.8 mm to (68.9, 55.5)
- moved J3 30.0 mm to (27.7, 79.0)
- moved R2 18.9 mm to (45.1, 31.3), turned to 180 degrees
- moved R1 18.3 mm to (45.0, 27.6), turned to 180 degrees
- moved SW2 17.7 mm to (49.1, 82.0), turned to 180 degrees
- moved J2 11.8 mm to (72.0, 27.7), turned to -90 degrees
- moved R4 8.49 mm to (76.1, 78.4), turned to 90 degrees
- moved D2 1.57 mm to (85.5, 65.7)
Connections:
- D2 pad 1: GND -> Net-(D2-K)
- R3 pad 2: 3.3V -> 5V
- R4 pad 1: Net-(D2-A) -> 3.3V
- R4 pad 2: Net-(R4-Pad2) -> MODOS
- SW1 pad 1: unconnected-(SW1-C-Pad1) -> 5V
- SW2 pad 1: MODOS -> 3.3V
- SW2 pad 2: Net-(R4-Pad2) -> GND
- U1 pad 12: DFPlayer2 -> unconnected-(U1-IO14-Pad12)
- U1 pad 13: DFPlayer1 -> unconnected-(U1-IO12-Pad13)
- U1 pad 27: unconnected-(U1-IO16-Pad27) -> DFPlayer1
- U1 pad 28: unconnected-(U1-IO17-Pad28) -> DFPlayer2
- U1 pad 33: unconnected-(U1-IO21-Pad33) -> SDA
- U1 pad 36: unconnected-(U1-IO22-Pad36) -> SCL
- U1 pad 7: SDA -> Net-(D2-A)
- U1 pad 8: SCL -> unconnected-(U1-IO33-Pad8)
Routing:
- net 5V: track 27.9 -> 113.0 mm
- net DFPlayer1: track 5.03 -> 40.8 mm
- net DFPlayer2: track 3.49 -> 31.2 mm
- net SDA: track 61.0 -> 47.8 mm
- net 3.3V: track 29.3 -> 41.6 mm
- net Net-(D2-A): track 15.1 -> 3.87 mm
- net Net-(R4-Pad2): track 10.9 -> 0.00 mm
- net RING1: track 13.3 -> 4.48 mm
- net SCL: track 49.4 -> 57.9 mm
- net Net-(U3-Rx): track 5.95 -> 14.3 mm
- net Net-(U3-Tx): track 5.17 -> 13.3 mm
- net TIP: track 9.11 -> 4.48 mm
- net Net-(D2-K): track 0.00 -> 4.58 mm
- net MODOS: track 11.6 -> 7.56 mm
- net Net-(D1-A): track 8.00 -> 4.50 mm

Commit message: Add files via upload
Parts:
- removed D2: LED, LED_THT:LED_Rectangular_W3.0mm_H2.0mm
- removed R5: 220, Resistor_THT:R_Axial_DIN0207_L6.3mm_D2.5mm_P7.62mm_Horizontal
- removed U1: ESP32-DEVKITC, HUELLAS:MODULE_ESP32-DEVKITC
- added D1: LED, LED_THT:LED_Rectangular_W3.0mm_H2.0mm, F.Cu at (138.9, 156.8)
- added D1: LED, LED_THT:LED_Rectangular_W3.0mm_H2.0mm, F.Cu at (62.6, 156.8)
- added D1: LED, LED_THT:LED_Rectangular_W3.0mm_H2.0mm, F.Cu at (214.5, 81.6)
- added D1: LED, LED_THT:LED_Rectangular_W3.0mm_H2.0mm, F.Cu at (216.1, 157.1)
- added D1: LED, LED_THT:LED_Rectangular_W3.0mm_H2.0mm, F.Cu at (137.3, 81.3)
- added D3: LED, LED_THT:LED_Rectangular_W3.0mm_H2.0mm, F.Cu at (177.8, 34.4)
- added D3: LED, LED_THT:LED_Rectangular_W3.0mm_H2.0mm, F.Cu at (100.6, 34.1)
- added D3: LED, LED_THT:LED_Rectangular_W3.0mm_H2.0mm, F.Cu at (26.0, 109.6)
- added D3: LED, LED_THT:LED_Rectangular_W3.0mm_H2.0mm, F.Cu at (179.5, 109.9)
- added D3: LED, LED_THT:LED_Rectangular_W3.0mm_H2.0mm, F.Cu at (102.3, 109.6)
- added D3: LED, LED_THT:LED_Rectangular_W3.0mm_H2.0mm, F.Cu at (24.3, 34.1)
- added G***: LOGO, HUELLAS:cardiotune, F.Cu at (155.7, 107.5)
- added G***: LOGO, HUELLAS:cardiotune, F.Cu at (154.1, 31.9)
- added G***: LOGO, HUELLAS:mollourtadopaty, F.Cu at (222.0, 33.1)
- added G***: LOGO, HUELLAS:mollourtadopaty, F.Cu at (146.5, 108.3)
- added G***: LOGO, HUELLAS:mollourtadopaty, F.Cu at (70.2, 108.3)
- added G***: LOGO, HUELLAS:cardiotune, F.Cu at (79.4, 107.5)
- added G***: LOGO, HUELLAS:mollourtadopaty, F.Cu at (144.8, 32.8)
- added G***: LOGO, HUELLAS:cardiotune, F.Cu at (231.3, 32.2)
- added G***: LOGO, HUELLAS:cardiotune, F.Cu at (232.9, 107.8)
- added G***: LOGO, HUELLAS:mollourtadopaty, F.Cu at (223.7, 108.6)
- added J1: TRRS, Connector_PinSocket_2.54mm:PinSocket_1x04_P2.54mm_Vertical, F.Cu at (134.9, 51.6)
- added J1: TRRS, Connector_PinSocket_2.54mm:PinSocket_1x04_P2.54mm_Vertical, F.Cu at (60.2, 127.2)
- added J1: TRRS, Connector_PinSocket_2.54mm:PinSocket_1x04_P2.54mm_Vertical, F.Cu at (136.5, 127.2)
- added J1: TRRS, Connector_PinSocket_2.54mm:PinSocket_1x04_P2.54mm_Vertical, F.Cu at (213.7, 127.5)
- added J1: TRRS, Connector_PinSocket_2.54mm:PinSocket_1x04_P2.54mm_Vertical, F.Cu at (212.1, 51.9)
- added J2: MAX30102, Connector_PinSocket_2.54mm:PinSocket_1x04_P2.54mm_Vertical, F.Cu at (99.8, 72.0)
- added J2: MAX30102, Connector_PinSocket_2.54mm:PinSocket_1x04_P2.54mm_Vertical, F.Cu at (177.0, 72.3)
- added J2: MAX30102, Connector_PinSocket_2.54mm:PinSocket_1x04_P2.54mm_Vertical, F.Cu at (178.7, 147.8)
- added J2: MAX30102, Connector_PinSocket_2.54mm:PinSocket_1x04_P2.54mm_Vertical, F.Cu at (25.2, 147.5)
- added J2: MAX30102, Connector_PinSocket_2.54mm:PinSocket_1x04_P2.54mm_Vertical, F.Cu at (101.5, 147.5)
- added J3: Screw_Terminal_01x02, TerminalBlock_Phoenix:TerminalBlock_Phoenix_MKDS-1,5-2-5.08_1x02_P5.08mm_Horizontal, F.Cu at (156.2, 82.9)
- added J3: Screw_Terminal_01x02, TerminalBlock_Phoenix:TerminalBlock_Phoenix_MKDS-1,5-2-5.08_1x02_P5.08mm_Horizontal, F.Cu at (157.9, 158.4)
- added J3: Screw_Terminal_01x02, TerminalBlock_Phoenix:TerminalBlock_Phoenix_MKDS-1,5-2-5.08_1x02_P5.08mm_Horizontal, F.Cu at (233.4, 83.2)
- added J3: Screw_Terminal_01x02, TerminalBlock_Phoenix:TerminalBlock_Phoenix_MKDS-1,5-2-5.08_1x02_P5.08mm_Horizontal, F.Cu at (235.1, 158.7)
- added J3: Screw_Terminal_01x02, TerminalBlock_Phoenix:TerminalBlock_Phoenix_MKDS-1,5-2-5.08_1x02_P5.08mm_Horizontal, F.Cu at (81.6, 158.4)
- added R1: 1K, Resistor_THT:R_Axial_DIN0207_L6.3mm_D2.5mm_P7.62mm_Horizontal, F.Cu at (225.1, 146.8)
- added R1: 1K, Resistor_THT:R_Axial_DIN0207_L6.3mm_D2.5mm_P7.62mm_Horizontal, F.Cu at (71.6, 146.5)
- added R1: 1K, Resistor_THT:R_Axial_DIN0207_L6.3mm_D2.5mm_P7.62mm_Horizontal, F.Cu at (147.9, 146.5)
- added R1: 1K, Resistor_THT:R_Axial_DIN0207_L6.3mm_D2.5mm_P7.62mm_Horizontal, F.Cu at (223.4, 71.3)
- added R1: 1K, Resistor_THT:R_Axial_DIN0207_L6.3mm_D2.5mm_P7.62mm_Horizontal, F.Cu at (146.2, 71.0)
- added R2: 1K, Resistor_THT:R_Axial_DIN0207_L6.3mm_D2.5mm_P7.62mm_Horizontal, F.Cu at (219.0, 71.4)
- added R2: 1K, Resistor_THT:R_Axial_DIN0207_L6.3mm_D2.5mm_P7.62mm_Horizontal, F.Cu at (67.2, 146.6)
- added R2: 1K, Resistor_THT:R_Axial_DIN0207_L6.3mm_D2.5mm_P7.62mm_Horizontal, F.Cu at (141.8, 71.1)
- added R2: 1K, Resistor_THT:R_Axial_DIN0207_L6.3mm_D2.5mm_P7.62mm_Horizontal, F.Cu at (220.7, 146.9)
- added R2: 1K, Resistor_THT:R_Axial_DIN0207_L6.3mm_D2.5mm_P7.62mm_Horizontal, F.Cu at (143.5, 146.6)
- added R3: 220, Resistor_THT:R_Axial_DIN0207_L6.3mm_D2.5mm_P7.62mm_Horizontal, F.Cu at (211.9, 78.1)
- added R3: 220, Resistor_THT:R_Axial_DIN0207_L6.3mm_D2.5mm_P7.62mm_Horizontal, F.Cu at (136.4, 153.3)
- added R3: 220, Resistor_THT:R_Axial_DIN0207_L6.3mm_D2.5mm_P7.62mm_Horizontal, F.Cu at (213.6, 153.6)
- added R3: 220, Resistor_THT:R_Axial_DIN0207_L6.3mm_D2.5mm_P7.62mm_Horizontal, F.Cu at (60.1, 153.3)
- added R3: 220, Resistor_THT:R_Axial_DIN0207_L6.3mm_D2.5mm_P7.62mm_Horizontal, F.Cu at (134.7, 77.8)
- added R4: 220, Resistor_THT:R_Axial_DIN0207_L6.3mm_D2.5mm_P7.62mm_Horizontal, F.Cu at (110.1, 41.5)
- added R4: 220, Resistor_THT:R_Axial_DIN0207_L6.3mm_D2.5mm_P7.62mm_Horizontal, F.Cu at (187.3, 41.8)
- added R4: 220, Resistor_THT:R_Axial_DIN0207_L6.3mm_D2.5mm_P7.62mm_Horizontal, F.Cu at (35.5, 117.0)
- added R4: 220, Resistor_THT:R_Axial_DIN0207_L6.3mm_D2.5mm_P7.62mm_Horizontal, F.Cu at (189.0, 117.3)
- added R4: 220, Resistor_THT:R_Axial_DIN0207_L6.3mm_D2.5mm_P7.62mm_Horizontal, F.Cu at (111.8, 117.0)
- added R6: 220, Resistor_THT:R_Axial_DIN0207_L6.3mm_D2.5mm_P7.62mm_Horizontal, F.Cu at (178.1, 100.2)
- added R6: 220, Resistor_THT:R_Axial_DIN0207_L6.3mm_D2.5mm_P7.62mm_Horizontal, F.Cu at (22.9, 24.4)
- added R6: 220, Resistor_THT:R_Axial_DIN0207_L6.3mm_D2.5mm_P7.62mm_Horizontal, F.Cu at (99.2, 24.4)
- added R6: 220, Resistor_THT:R_Axial_DIN0207_L6.3mm_D2.5mm_P7.62mm_Horizontal, F.Cu at (176.4, 24.7)
- added R6: 220, Resistor_THT:R_Axial_DIN0207_L6.3mm_D2.5mm_P7.62mm_Horizontal, F.Cu at (100.9, 99.9)
- added R6: 220, Resistor_THT:R_Axial_DIN0207_L6.3mm_D2.5mm_P7.62mm_Horizontal, F.Cu at (24.6, 99.9)
- added SW1: SW_Nidec_CAS-120A1, Connector_PinSocket_2.54mm:PinSocket_1x02_P2.54mm_Vertical, F.Cu at (224.4, 153.6)
- added SW1: SW_Nidec_CAS-120A1, Connector_PinSocket_2.54mm:PinSocket_1x02_P2.54mm_Vertical, F.Cu at (145.5, 77.8)
- added SW1: SW_Nidec_CAS-120A1, Connector_PinSocket_2.54mm:PinSocket_1x02_P2.54mm_Vertical, F.Cu at (70.9, 153.3)
- added SW1: SW_Nidec_CAS-120A1, Connector_PinSocket_2.54mm:PinSocket_1x02_P2.54mm_Vertical, F.Cu at (147.2, 153.3)
- added SW1: SW_Nidec_CAS-120A1, Connector_PinSocket_2.54mm:PinSocket_1x02_P2.54mm_Vertical, F.Cu at (222.7, 78.1)
- added SW2: SW_Push, Button_Switch_THT:SW_PUSH_6mm, F.Cu at (116.6, 28.2)
- added SW2: SW_Push, Button_Switch_THT:SW_PUSH_6mm, F.Cu at (118.2, 103.8)
- added SW2: SW_Push, Button_Switch_THT:SW_PUSH_6mm, F.Cu at (195.4, 104.0)
- added SW2: SW_Push, Button_Switch_THT:SW_PUSH_6mm, F.Cu at (193.8, 28.5)
- added SW2: SW_Push, Button_Switch_THT:SW_PUSH_6mm, F.Cu at (42.0, 103.8)
- added U2: ESP32-DEVKIT-V1, RF_Module:MODULE_ESP32_DEVKIT_V1, F.Cu at (197.0, 132.8)
- added U2: ESP32-DEVKIT-V1, RF_Module:MODULE_ESP32_DEVKIT_V1, F.Cu at (195.3, 57.3)
- added U2: ESP32-DEVKIT-V1, RF_Module:MODULE_ESP32_DEVKIT_V1, F.Cu at (118.1, 57.0)
- added U2: ESP32-DEVKIT-V1, RF_Module:MODULE_ESP32_DEVKIT_V1, F.Cu at (119.8, 132.5)
- added U2: ESP32-DEVKIT-V1, RF_Module:MODULE_ESP32_DEVKIT_V1, F.Cu at (41.8, 57.0)
- added U2: ESP32-DEVKIT-V1, RF_Module:MODULE_ESP32_DEVKIT_V1, F.Cu at (43.5, 132.5)
- added U3: ~, HUELLAS:MODULE_DFR0299, F.Cu at (147.8, 50.4)
- added U3: ~, HUELLAS:MODULE_DFR0299, F.Cu at (226.7, 126.2)
- added U3: ~, HUELLAS:MODULE_DFR0299, F.Cu at (73.2, 125.9)
- added U3: ~, HUELLAS:MODULE_DFR0299, F.Cu at (225.0, 50.7)
- added U3: ~, HUELLAS:MODULE_DFR0299, F.Cu at (149.5, 125.9)
- SW1: footprint Connector_PinHeader_2.54mm:PinHeader_2x01_P2.54mm_Vertical -> Connector_PinSocket_2.54mm:PinSocket_1x02_P2.54mm_Vertical
- moved J2 65.7 mm to (23.5, 72.0), turned to 180 degrees
- moved R4 56.1 mm to (33.8, 41.5), turned to -90 degrees
- moved SW2 54.4 mm to (40.3, 28.2)
- moved J3 52.4 mm to (79.9, 82.9), turned to 90 degrees
- moved R1 50.1 mm to (69.9, 71.0), turned to 90 degrees
- moved G*** 44.8 mm to (77.8, 31.9)
- moved R2 44.8 mm to (65.5, 71.1), turned to 90 degrees
- moved G*** 41.0 mm to (68.5, 32.8)
- moved SW1 39.6 mm to (69.2, 77.8), turned to 90 degrees
- moved D1 36.8 mm to (61.0, 81.3), turned to 180 degrees
- moved J1 33.5 mm to (58.6, 51.6), turned to 180 degrees
- moved U3 30.7 mm to (71.5, 50.4)
- moved R3 28.6 mm to (58.4, 77.8), turned to 0 degrees
Connections:
- J1 pad 1: GND -> TIP LEFT
- J1 pad 2: unconnected-(J1-Pin_2-Pad2) -> RING RIGHT
- J1 pad 3: RING1 -> GND
- J1 pad 4: TIP -> unconnected-(J1-Pin_4-Pad4)
- U3 pad 4: RING1 -> RING RIGHT
- U3 pad 5: TIP -> TIP LEFT
Routing:
- net 5V: track 113.0 -> 712.5 mm
- net DFPlayer1: track 40.8 -> 180.3 mm
- net Net-(U3-Rx): track 14.3 -> 152.7 mm
- net DFPlayer2: track 31.2 -> 144.9 mm
- net 3.3V: track 41.6 -> 146.5 mm
- net Net-(U3-Tx): track 13.3 -> 114.6 mm
- net MODOS: track 7.56 -> 96.9 mm
- net Net-(D3-A): track 0.00 -> 85.2 mm
- net Net-(D3-K): track 0.00 -> 61.5 mm
- net Net-(J3-Pin_2): track 7.85 -> 48.8 mm
- net TIP LEFT: track 0.00 -> 23.8 mm
- net RING RIGHT: track 0.00 -> 23.8 mm
- net Net-(D1-A): track 4.50 -> 21.0 mm
- net SDA: track 47.8 -> 33.6 mm
- net Net-(D2-K): track 4.58 -> 0.00 mm
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